Commit message: Use file:// mesh URIs and add gui:=false to gazebo_world
package:// meshes needed the ROS share dir on GAZEBO_MODEL_PATH, which
made gzclient log a Missing model.config error for every folder there.
file://jetbot_ros
jetbot_ros/__init__.py
jetbot_ros/motors_nvidia.py
jetbot_ros/dnn
jetbot_ros/dnn/__init__.py
jetbot_ros/dnn/reshape_model.py
jetbot_ros/dnn/xy_dataset.py
jetbot_ros/dnn/__pycache__
jetbot_ros/dnn/__pycache__/__init__.cpython-310.pyc
jetbot_ros/dnn/__pycache__/navigation_model.cpython-310.pyc
jetbot_ros/dnn/train.py
jetbot_ros/dnn/navigation_model.py
jetbot_ros/nav_model.py
jetbot_ros/oled.py
jetbot_ros/teleop_keyboard.py
jetbot_ros/motors_waveshare.py
jetbot_ros/data_collection.py
jetbot_ros/__pycache__
jetbot_ros/__pycache__/__init__.cpython-310.pyc
jetbot_ros/__pycache__/gazebo_spawn.cpython-310.pyc
jetbot_ros/__pycache__/teleop_keyboard.cpython-310.pyc
jetbot_ros/__pycache__/nav_model.cpython-310.pyc
jetbot_ros/gazebo_spawn.py
jetbot_ros/motors.py
jetbot_ros/motors_sparkfun.py
jetbot_ros/oled_ssd1306.py resolves in both Gazebo classic and RViz2, so
drop that and spawn_entity's -package_to_model. gui:=false runs gzserver
only, for headless checks and machines without a display.

Co-Authored-By: Claude Fable 5.1 <noreply@anthropic.com>

File: urdf/jetbot.urdf.xacro (robot description, xacro)
@@ -12,5 +12,7 @@
 -->
 <robot xmlns:xacro="http://www.ros.org/wiki/xacro" name="jetbot">
-  <xacro:property name="mesh_dir"   value="package://jetbot_ros/models/jetbot/meshes"/>
+  <!-- file:// works for both RViz2 and Gazebo classic; package:// would need the ROS share dir on
+       GAZEBO_MODEL_PATH, which makes gzclient's Insert panel complain about every non-model folder there -->
+  <xacro:property name="mesh_dir"   value="file://$(find jetbot_ros)/models/jetbot/meshes"/>
   <xacro:property name="mesh_scale" value="0.001 0.001 0.001"/>
   <xacro:property name="mesh_rpy"   value="${pi/2} 0 ${pi/2}"/>
